Commit message: todo good?

File: test1week11/practice/l4_ws/install/robot_description/share/robot_description/urdf/indice.urdf (robot description, URDF)
Before this commit: robot example_robot_visible, 11 links, 10 joints
Links:
- removed link link0_passive
- removed link link0_x_axis
- removed link link1
- removed link link1_passive
- removed link link1_x_axis
- removed link link2
- removed link link2_passive
- removed link link2_x_axis
- removed link link3
- removed link link3_passive
- removed link link3_x_axis
- added link r1_link0_passive; visual origin rpy=0 0 0 xyz=0 0 0
- added link r1_link0_x_axis; visual origin rpy=0 0 0 xyz=0 0 0
- added link r1_link1
- added link r1_link1_passive; visual cylinder length=2.0 radius=0.05
- added link r1_link1_x_axis; visual cylinder length=0.05 radius=0.005
- added link r1_link2
- added link r1_link2_passive; visual cylinder length=1.5 radius=0.05
- added link r1_link2_x_axis; visual cylinder length=0.05 radius=0.005
- added link r1_link3
- added link r1_link3_passive; visual cylinder length=0.8 radius=0.05
- added link r1_link3_x_axis; visual cylinder length=0.05 radius=0.005
- added link r2_link0_passive; visual origin rpy=0 0 0 xyz=0 0 0
- added link r2_link0_x_axis; visual origin rpy=0 0 0 xyz=0 0 0
- added link r2_link1
- added link r2_link1_passive; visual cylinder length=0.5 radius=0.05
- added link r2_link1_x_axis; visual cylinder length=0.5 radius=0.05
- added link r2_link2
- added link r2_link2_passive; visual cylinder length=0.5 radius=0.05
- added link r2_link2_x_axis; visual cylinder length=0.5 radius=0.05
- added link r2_link3
- added link r2_link3_passive; visual cylinder length=0.5 radius=0.05
- added link r2_link3_x_axis; visual cylinder length=0.5 radius=0.05
- added link world
Joints:
- removed joint q0_x
- removed joint q1
- removed joint q1_passive
- removed joint q1_x
- removed joint q2
- removed joint q2_passive
- removed joint q2_x
- removed joint q3
- removed joint q3_passive
- removed joint q3_x
- added joint r1_q0_x: type fixed, parent r1_link0_passive, child r1_link0_x_axis, origin xyz=0 0 0 rpy=0 1.571 0
- added joint r1_q1: type revolute, parent r1_link0_passive, child r1_link1, origin xyz=0 0 0.1 rpy=0 0 0, axis 0 0 1, limit lower=-1.5 upper=1.5 effort=411 velocity=1.57
- added joint r1_q1_passive: type fixed, parent r1_link1, child r1_link1_passive, origin xyz=2 0 0 rpy=0 0 0
- added joint r1_q1_x: type fixed, parent r1_link1_passive, child r1_link1_x_axis, origin xyz=0 0 0 rpy=0 1.571 0
- added joint r1_q2: type revolute, parent r1_link1_passive, child r1_link2, origin xyz=0 0 0 rpy=0 0 0, axis 0 0 1, limit lower=-1.5 upper=1.5 effort=411 velocity=1.57
- added joint r1_q2_passive: type fixed, parent r1_link2, child r1_link2_passive, origin xyz=1.5 0 0 rpy=0 0 0
- added joint r1_q2_x: type fixed, parent r1_link2_passive, child r1_link2_x_axis, origin xyz=0 0 0 rpy=0 1.571 0
- added joint r1_q3: type revolute, parent r1_link2_passive, child r1_link3, origin xyz=0 0 0 rpy=0 0 0, axis 0 0 1, limit lower=-1.5 upper=1.5 effort=411 velocity=1.57
- added joint r1_q3_passive: type fixed, parent r1_link3, child r1_link3_passive, origin xyz=0.8 0 0 rpy=0 0 0
- added joint r1_q3_x: type fixed, parent r1_link3_passive, child r1_link3_x_axis, origin xyz=0 0 0 rpy=0 1.571 0
- added joint r2_q0_x: type fixed, parent r2_link0_passive, child r2_link0_x_axis, origin xyz=0 0 0 rpy=0 1.571 0
- added joint r2_q1: type revolute, parent r2_link0_passive, child r2_link1, origin xyz=0 0 0.5 rpy=0 0 0, axis 1 0 0, limit lower=-2.9671 upper=2.9671 effort=87 velocity=2.1750
- added joint r2_q1_passive: type fixed, parent r2_link1, child r2_link1_passive, origin xyz=0 0 0 rpy=1.5707963267948966 0 0
- added joint r2_q1_x: type fixed, parent r2_link1_passive, child r2_link1_x_axis, origin xyz=0 0 0 rpy=0 1.571 0
- added joint r2_q2: type revolute, parent r2_link1_passive, child r2_link2, origin xyz=0 0 0 rpy=0 0 0, axis 0 0 1, limit lower=-2.9671 upper=2.9671 effort=87 velocity=2.1750
- added joint r2_q2_passive: type fixed, parent r2_link2, child r2_link2_passive, origin xyz=1.3 0 0 rpy=0 0 0
- added joint r2_q2_x: type fixed, parent r2_link2_passive, child r2_link2_x_axis, origin xyz=0 0 0 rpy=0 1.571 0
- added joint r2_q3: type revolute, parent r2_link2_passive, child r2_link3, origin xyz=0 0 0 rpy=0 0 0, axis 0 0 1, limit lower=-2.9671 upper=2.9671 effort=87 velocity=2.1750
- added joint r2_q3_passive: type fixed, parent r2_link3, child r2_link3_passive, origin xyz=0.9 0 0 rpy=0 0 0
- added joint r2_q3_x: type fixed, parent r2_link3_passive, child r2_link3_x_axis, origin xyz=0 0 0 rpy=0 1.571 0
- added joint world_to_r1: type fixed, parent world, child r1_link0_passive, origin xyz=0 0 0 rpy=0 0 0
- added joint world_to_r2: type fixed, parent world, child r2_link0_passive, origin xyz=3 0 0 rpy=0 0 0
